Commit message: Rebase from 'release/hydro/r2_description'

File: robots/r2_fullbody.urdf.xacro (robot description, xacro)
@@ -1,6 +1,6 @@
 <?xml version="1.0" ?>
-  <robot xmlns:xacro="http://wiki.ros.org/xacro" name="r2c_full_body" >
+  <robot xmlns:xacro="http://wiki.ros.org/xacro" name="r2_fullbody" >
   <link name="world"/>
-  <property name="robot_name" value= "/r2/" />
+  <property name="robot_name" value= "r2/" />
 <!--  transforms in first joint don't seem to work properly-->
   <joint name="${robot_name}fixed/world/robot_world" type="fixed">
@@ -9,7 +9,4 @@
     <origin rpy="0 0 0.0" xyz="0.0 0.0 0.0"/>
   </joint>
-  <xacro:include filename="$(find r2_description)/robots/r2c_full_body_no_world.urdf.xacro" />
-  <xacro:robot_base_origin>
-    <origin xyz="0 0 1.4" rpy="0 0 0" />
-  </xacro:robot_base_origin>
+  <xacro:include filename="$(find r2_description)/robots/r2_fullbody_no_world.urdf.xacro" />
 </robot>

File: robots/r2_fullbody_no_world.urdf.xacro (robot description, xacro)
@@ -1,14 +1,12 @@
 <?xml version="1.0" ?>
-<robot name="r2c_full_body" xmlns:xacro="http://wiki.ros.org/xacro">
-  <property name="robot_name" value= "/r2/" />
-  <non_visual_link name="${robot_name}robot_world"/>
-  <xacro:macro name="robot_base_origin" params="*origin">
-    <joint name="${robot_name}fixed/robot_world/robot_base" type="fixed">
+<robot name="r2" xmlns:xacro="http://playerstage.sourceforge.net/gazebo/xmlschema/#interface">
+  <property name="robot_name" value= "r2/" />
+  <link name="${robot_name}robot_world"/>
+  <joint name="${robot_name}fixed/robot_world/robot_base" type="fixed">
       <parent link="${robot_name}robot_world"/>
       <child link="${robot_name}robot_base"/>
-      <xacro:insert_block name="origin" />
-    </joint>
-  </xacro:macro>
-  <non_visual_link name="${robot_name}robot_base"/>
+      <origin rpy="0 3.14159 1.57079" xyz="0.255 0.9 1.365"/>
+  </joint>
+  <link name="${robot_name}robot_base"/>
   <joint name="${robot_name}fixed/robot_base/leg_stand_connection" type="fixed">
     <parent link="${robot_name}robot_base"/>
@@ -24,8 +22,8 @@
   <xacro:include filename="$(find r2_description)/urdf/r2.right_arm.xacro" />
   <xacro:include filename="$(find r2_description)/urdf/r2.right_hand.xacro" />
-  <xacro:include filename="$(find r2_description)/urdf/r2c_legs/r2c_legs.pelvis.xacro" />
-  <xacro:include filename="$(find r2_description)/urdf/r2c_legs/r2c_legs.left_leg.xacro" />
-  <xacro:include filename="$(find r2_description)/urdf/r2c_legs/r2c_legs.left_foot.xacro" />
-  <xacro:include filename="$(find r2_description)/urdf/r2c_legs/r2c_legs.right_leg.xacro" />
-  <xacro:include filename="$(find r2_description)/urdf/r2c_legs/r2c_legs.right_foot.xacro" />
+  <xacro:include filename="$(find r2_description)/urdf/r2_legs/r2_legs.pelvis.xacro" />
+  <xacro:include filename="$(find r2_description)/urdf/r2_legs/r2_legs.left_leg.xacro" />
+  <xacro:include filename="$(find r2_description)/urdf/r2_legs/r2_legs.left_foot.xacro" />
+  <xacro:include filename="$(find r2_description)/urdf/r2_legs/r2_legs.right_leg.xacro" />
+  <xacro:include filename="$(find r2_description)/urdf/r2_legs/r2_legs.right_foot.xacro" />
 </robot>

File: urdf/r2_legs/r2_legs.left_foot.xacro (robot description, xacro)
@@ -15,19 +15,31 @@
     <inertial>
       <mass value="4.40475"/>
-      <inertia ixx="0.04809" ixy="0.00026" ixz="0.00038" iyy="0.04403" iyz="-0.00321" izz="0.0127"/>
+      <inertia ixx="0.1" ixy="0.0" ixz="0.0" iyy="0.1" iyz="0.0" izz="0.1"/>
     </inertial>
     <visual>
       <geometry>
-        <mesh filename="package://r2_description/meshes/r2c_legs/r2cl_foot.dae"/>
+        <mesh filename="package://r2_description/meshes/r2_legs/r2cl_foot.dae"/>
       </geometry>
-      <origin rpy="0 0 0" xyz="0 0 0"/>
+      <origin xyz="0 0 0" rpy="0 0 0" />
     </visual>
     <collision>
       <geometry>
-        <mesh filename="package://r2_description/meshes/r2c_legs/r2cl_foot.dae"/>
+        <mesh filename="package://r2_description/meshes/r2_legs/r2cl_foot.dae"/>
       </geometry>
       <origin rpy="0 0 0" xyz="0 0 0"/>
     </collision>
   </link>
+  <joint name="${robot_name}fixed/left_foot/simulated_camboard" type="fixed">
+    <parent link="${robot_name}left_leg_foot"/>
+    <child link="${robot_name}simulated_left_foot_camboard_frame"/>
+    <dynamics damping="1.0" />
+    <origin rpy="0 -1.57 -1.57" xyz="0.015 0.07 .165"/>
+  </joint>
+  <joint name="${robot_name}fixed/left_foot/simulated_camboard_depth" type="fixed">
+    <parent link="${robot_name}left_leg_foot"/>
+    <child link="${robot_name}simulated_left_foot_camboard_depth_frame"/>
+    <dynamics damping="1.0" />
+    <origin rpy="3.14 3.14 0" xyz="0.015 0.07 .165"/>
+  </joint>
 <!--  placeholder for screw joint-->
   <joint name="${robot_name}left_leg/gripper/joint0" type="revolute">
@@ -79,12 +91,26 @@
   <non_visual_link name="${robot_name}left_hr_tip"/>
   <non_visual_link name="${robot_name}left_st_tip"/>
+ <!-- simulated camboard -->
+  <link name="${robot_name}simulated_left_foot_camboard_frame">
+    <inertial>
+      <mass value=".1"/>
+      <inertia ixx=".01" ixy="0.0" ixz="0.0" iyy=".01" iyz="0.0" izz=".01"/>
+    </inertial>
+  </link>
+  <!-- simulated camboard -->
+  <link name="${robot_name}simulated_left_foot_camboard_depth_frame">
+    <inertial>
+      <mass value=".1"/>
+      <inertia ixx=".01" ixy="0.0" ixz="0.0" iyy=".01" iyz="0.0" izz=".01"/>
+    </inertial>
+  </link>
   <link name="${robot_name}left_leg_jaw0">
     <inertial>
       <mass value="0.16268"/>
-      <inertia ixx="0.001" ixy="0.0" ixz="0.0" iyy="0.001" iyz="0.0" izz="0.001"/>
+      <inertia ixx="0.1" ixy="0.0" ixz="0.0" iyy="0.1" iyz="0.0" izz="0.1"/>
     </inertial>
     <visual>
       <geometry>
-        <mesh filename="package://r2_description/meshes/r2c_legs/r2cl_foot_jaw1.dae"/>
+        <mesh filename="package://r2_description/meshes/r2_legs/r2cl_foot_jaw1.dae"/>
       </geometry>
       <origin rpy="0 0 0" xyz="0 0 0"/>
@@ -92,5 +118,5 @@
     <collision>
       <geometry>
-        <mesh filename="package://r2_description/meshes/r2c_legs/r2cl_foot_jaw1.dae"/>
+        <mesh filename="package://r2_description/meshes/r2_legs/r2cl_foot_jaw1.dae"/>
       </geometry>
       <origin rpy="0 0 0" xyz="0 0 0"/>
@@ -100,9 +126,9 @@
     <inertial>
       <mass value="0.16268"/>
-      <inertia ixx="0.001" ixy="0.0" ixz="0.0" iyy="0.001" iyz="0.0" izz="0.001"/>
+      <inertia ixx="0.1" ixy="0.0" ixz="0.0" iyy="0.1" iyz="0.0" izz="0.1"/>
     </inertial>
     <visual>
       <geometry>
-        <mesh filename="package://r2_description/meshes/r2c_legs/r2cl_foot_jaw2.dae"/>
+        <mesh filename="package://r2_description/meshes/r2_legs/r2cl_foot_jaw2.dae"/>
       </geometry>
       <origin rpy="0 0 0" xyz="0 0 0"/>
@@ -110,5 +136,5 @@
     <collision>
       <geometry>
-        <mesh filename="package://r2_description/meshes/r2c_legs/r2cl_foot_jaw2.dae"/>
+        <mesh filename="package://r2_description/meshes/r2_legs/r2cl_foot_jaw2.dae"/>
       </geometry>
       <origin rpy="0 0 0" xyz="0 0 0"/>

File: urdf/r2_legs/r2_legs.right_foot.xacro (robot description, xacro)
@@ -15,20 +15,32 @@
     <inertial>
       <mass value="4.40475"/>
-      <inertia ixx="0.04809" ixy="0.00026" ixz="0.00038" iyy="0.04403" iyz="-0.00321" izz="0.0127"/>
+       <inertia ixx="0.1" ixy="0.0" ixz="0.0" iyy="0.1" iyz="0.0" izz="0.1"/>
     </inertial>
     <visual>
       <geometry>
-        <mesh filename="package://r2_description/meshes/r2c_legs/r2cl_foot.dae"/>
+        <mesh filename="package://r2_description/meshes/r2_legs/r2cl_foot.dae"/>
       </geometry>
       <material name="gold"/>
-      <origin rpy="0 0 0" xyz="0 0 0"/>
+      <origin xyz="0 0 0" rpy="0 0 0" />
     </visual>
     <collision>
       <geometry>
-        <mesh filename="package://r2_description/meshes/r2c_legs/r2cl_foot.dae"/>
+        <mesh filename="package://r2_description/meshes/r2_legs/r2cl_foot.dae"/>
       </geometry>
       <origin rpy="0 0 0" xyz="0 0 0"/>
     </collision>
   </link>
+  <joint name="${robot_name}fixed/right_foot/simulated_camboard" type="fixed">
+    <parent link="${robot_name}right_leg_foot"/>
+    <child link="${robot_name}simulated_right_foot_camboard_frame"/>
+    <dynamics damping="1.0" />
+    <origin rpy="0 -1.57 -1.57" xyz="0.015 0.07 .165"/>
+  </joint>
+  <joint name="${robot_name}fixed/right_foot/simulated_camboard_depth" type="fixed">
+    <parent link="${robot_name}right_leg_foot"/>
+    <child link="${robot_name}simulated_right_foot_camboard_depth_frame"/>
+    <dynamics damping="1.0" />
+    <origin rpy="3.14 3.14 0" xyz="0.015 0.07 .165"/>
+  </joint>
 <!--  placeholder for screw joint-->
   <joint name="${robot_name}right_leg/gripper/joint0" type="prismatic">
@@ -82,12 +94,26 @@
   <non_visual_link name="${robot_name}right_hr_tip"/>
   <non_visual_link name="${robot_name}right_st_tip"/>
+  <!-- simulated camboard -->
+  <link name="${robot_name}simulated_right_foot_camboard_frame">
+    <inertial>
+      <mass value=".1"/>
+      <inertia ixx=".01" ixy="0.0" ixz="0.0" iyy=".01" iyz="0.0" izz=".01"/>
+    </inertial>
+  </link>
+  <!-- simulated camboard -->
+  <link name="${robot_name}simulated_right_foot_camboard_depth_frame">
+    <inertial>
+      <mass value=".1"/>
+      <inertia ixx=".01" ixy="0.0" ixz="0.0" iyy=".01" iyz="0.0" izz=".01"/>
+    </inertial>
+  </link>
   <link name="${robot_name}right_leg_jaw0">
     <inertial>
       <mass value="0.16268"/>
-      <inertia ixx="0.001" ixy="0.0" ixz="0.0" iyy="0.001" iyz="0.0" izz="0.001"/>
+      <inertia ixx="0.1" ixy="0.0" ixz="0.0" iyy="0.1" iyz="0.0" izz="0.1"/>
     </inertial>
     <visual>
       <geometry>
-        <mesh filename="package://r2_description/meshes/r2c_legs/r2cl_foot_jaw1.dae"/>
+        <mesh filename="package://r2_description/meshes/r2_legs/r2cl_foot_jaw1.dae"/>
       </geometry>
       <origin rpy="0 0 0" xyz="0 0 0"/>
@@ -95,5 +121,5 @@
     <collision>
       <geometry>
-        <mesh filename="package://r2_description/meshes/r2c_legs/r2cl_foot_jaw1.dae"/>
+        <mesh filename="package://r2_description/meshes/r2_legs/r2cl_foot_jaw1.dae"/>
       </geometry>
       <origin rpy="0 0 0" xyz="0 0 0"/>
@@ -103,9 +129,9 @@
     <inertial>
       <mass value="0.16268"/>
-      <inertia ixx="0.001" ixy="0.0" ixz="0.0" iyy="0.001" iyz="0.0" izz="0.001"/>
+      <inertia ixx="0.1" ixy="0.0" ixz="0.0" iyy="0.1" iyz="0.0" izz="0.1"/>
     </inertial>
     <visual>
       <geometry>
-        <mesh filename="package://r2_description/meshes/r2c_legs/r2cl_foot_jaw2.dae"/>
+        <mesh filename="package://r2_description/meshes/r2_legs/r2cl_foot_jaw2.dae"/>
       </geometry>
       <origin rpy="0 0 0" xyz="0 0 0"/>
@@ -113,5 +139,5 @@
     <collision>
       <geometry>
-        <mesh filename="package://r2_description/meshes/r2c_legs/r2cl_foot_jaw2.dae"/>
+        <mesh filename="package://r2_description/meshes/r2_legs/r2cl_foot_jaw2.dae"/>
       </geometry>
       <origin rpy="0 0 0" xyz="0 0 0"/>
